File: Hardware/Advanced Flight Computer.kicad_pcb (KiCad board)
At the start: 4 copper layers, 65 x 110 mm, 163 parts, among them CN1 ATGM336H-6N-74, J1 Conn_01x03_Pin, J2 Conn_01x04_Pin, J3 Conn_01x02_Pin, J4 Conn_01x02_Pin, J5 Conn_01x02_Pin, J6 Conn_01x02_Pin, M1 Motor_Servo, M2 Motor_Servo, M3 Motor_Servo, M4 Motor_Servo, M5 Motor_Servo, M6 Motor_Servo, P1 WJ500V-5.08-2P-14-00A, P2 WJ500V-5.08-2P-14-00A, P3 WJ500V-5.08-2P-14-00A, P4 WJ500V-5.08-2P-14-00A, P5 WJ500V-5.08-2P-14-00A, P6 WJ500V-5.08-2P-14-00A, P7 WJ500V-5.08-2P-14-00A, P8 WJ500V-5.08-2P-14-00A, Q1 IRLML6402_C518785, Q10 2N7002LT1G, Q11 2N7002LT1G, Q12 IRLML6402_C518785, Q13 2N7002LT1G, Q2 IRLML6402_C518785, Q3 2N7002LT1G, Q4 IRLML6402_C518785, Q5 2N7002LT1G, Q6 IRLML6402_C518785, Q7 2N2222AU, Q8 2N7002LT1G, Q9 IRLML6402_C518785, SW1 TS-1088-AR02016, SW2 TS-1088-AR02016, U1 BMP580, U10 0438006.WRGT, U11 0438006.WRGT, U12 0438006.WRGT, U13 0438006.WRGT, U2 STM32H743VITx, U3 ICM-45686, U4 LMR51430XDDCR, U5 AP64501SP-13, U6 RA-02, U7 TPS2121RUXR, U8 0438006.WRGT, U9 0438006.WRGT, X1 X322525MOB4SI, X2 Q13FC1350000400

Commit message: Update with latest changes
Parts:
- added SWD: Conn_01x05_Pin, Connector_PinHeader_2.54mm:PinHeader_1x05_P2.54mm_Vertical, F.Cu at (101.1, 52.5)
- C1, C10, C11, C12, C13, C2, C25, C27, C3, C32, C33, C4, C5, C6, C7, C8, C9, R19, R20, R3, R4, R5, R6, R7, U4, U5, U7: moved to F.Cu
- moved R3 15.0 mm to (48.3, 122.7), turned to 90 degrees
- moved C4 12.9 mm to (62.0, 116.6), turned to 90 degrees
- moved R4 11.7 mm to (51.7, 123.6), turned to 180 degrees
- moved C1 11.3 mm to (48.0, 119.7), turned to 90 degrees
- moved R20 10.0 mm to (55.8, 112.4), turned to 90 degrees
- moved C3 9.42 mm to (59.5, 116.6), turned to 90 degrees
- moved R19 8.81 mm to (56.8, 114.3), turned to -90 degrees
- moved U4 8.45 mm to (51.5, 121.1), turned to -90 degrees
- moved R5 8.41 mm to (62.8, 126.6), turned to -90 degrees
- moved C12 7.98 mm to (54.6, 137.0)
- moved C7 7.57 mm to (52.8, 129.4)
- moved C27 7.24 mm to (54.0, 112.6), turned to 0 degrees
- moved C6 7.22 mm to (50.1, 136.7)
- moved C11 7.22 mm to (69.2, 127.5), turned to 90 degrees
- moved C10 7.00 mm to (67.0, 127.5)
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- renumbered U6 to LORA
Connections:
- U2 pad 72: unconnected-(U2-PA13-Pad72) -> /SWDIO
- U2 pad 76: unconnected-(U2-PA14-Pad76) -> /SWCLK
Routing:
- net /RESET: track 29.4 -> 102.7 mm, vias 2 -> 3
- net /SWCLK: track 0.00 -> 70.6 mm
- net /SWDIO: track 0.00 -> 39.7 mm
- net Net-(C12-Pad1): track 1.78 -> 12.2 mm, vias 0 -> 2
- net /POWER_ST: track 65.3 -> 55.3 mm, vias 4 -> 3
- net +BATT: track 198.6 -> 189.5 mm
- net +5V: track 181.5 -> 172.6 mm, vias 8 -> 7
- net /I2C_SCL: track 85.3 -> 93.6 mm
- net +3.3V: track 105.7 -> 97.5 mm, vias 23 -> 25
- net Net-(U5-FB): track 12.5 -> 20.0 mm
- net VBUS: track 78.2 -> 70.9 mm, vias 3 -> 7
- net GND: track 223.3 -> 217.3 mm, vias 65 -> 72
- net /BUZZER: track 41.8 -> 36.2 mm
- net Net-(U5-SW): track 7.85 -> 11.7 mm, vias 1 -> 0
- net Net-(U4-SW): track 11.6 -> 14.3 mm, vias 2 -> 3
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- added copper zone on B.Cu, net +3.3V
- added copper zone on F.Cu, net GND
- added copper zone on In1.Cu, net GND
- removed copper zone on In1.Cu, net +3.3V
