File: Hardware/Advanced Flight Computer.kicad_pcb (KiCad board)
At the start: 4 copper layers, 65 x 110 mm, 164 parts, among them CN1 ATGM336H-6N-74, J1 Conn_01x03_Pin, J2 Conn_01x04_Pin, J3 Conn_01x02_Pin, J4 Conn_01x02_Pin, J5 Conn_01x02_Pin, J6 Conn_01x02_Pin, M1 Motor_Servo, M2 Motor_Servo, M3 Motor_Servo, M4 Motor_Servo, M5 Motor_Servo, M6 Motor_Servo, P1 WJ500V-5.08-2P-14-00A, P2 WJ500V-5.08-2P-14-00A, P3 WJ500V-5.08-2P-14-00A, P4 WJ500V-5.08-2P-14-00A, P5 WJ500V-5.08-2P-14-00A, P6 WJ500V-5.08-2P-14-00A, P7 WJ500V-5.08-2P-14-00A, P8 WJ500V-5.08-2P-14-00A, Q1 IRLML6402_C518785, Q10 2N7002LT1G, Q11 2N7002LT1G, Q12 IRLML6402_C518785, Q13 2N7002LT1G, Q2 IRLML6402_C518785, Q3 2N7002LT1G, Q4 IRLML6402_C518785, Q5 2N7002LT1G, Q6 IRLML6402_C518785, Q7 2N2222AU, Q8 2N7002LT1G, Q9 IRLML6402_C518785, SW1 TS-1088-AR02016, SW2 TS-1088-AR02016, U1 BMP580, U10 0438006.WRGT, U11 0438006.WRGT, U12 0438006.WRGT, U13 0438006.WRGT, U2 STM32H743VITx, U3 ICM-45686, U4 LMR51430XDDCR, U5 AP64501SP-13, U7 TPS2121RUXR, U8 0438006.WRGT, U9 0438006.WRGT, X1 X322525MOB4SI, X2 Q13FC1350000400

Commit message: Update with latest changes
Parts:
- removed Q10, Q11, Q13, Q5, Q8: 2N7002LT1G, lcsc:SOT-23_L2.9-W1.3-P1.90-LS2.4-BR
- removed Q12, Q4, Q6, Q9: IRLML6402_C518785, lcsc:SOT-23-3_L2.9-W1.3-P1.90-LS2.4-BR
- removed R44, R48: 100k, Resistor_SMD:R_0402_1005Metric
- removed R45, R49: 10k, Resistor_SMD:R_0201_0603Metric
- removed R46: 1k, Resistor_SMD:R_0201_0603Metric
- removed R47: 100, Resistor_SMD:R_0201_0603Metric
- Q1, Q2: value IRLML6402_C518785 -> SI7232DN-T1-GE3; footprint lcsc:SOT-23-3_L2.9-W1.3-P1.90-LS2.4-BR -> lcsc:POWER-1212-8_L3.3-W3.3-P0.66-LS3.3-BL
- Q3: value 2N7002LT1G -> SI7232DN-T1-GE3; footprint lcsc:SOT-23_L2.9-W1.3-P1.90-LS2.4-BR -> lcsc:POWER-1212-8_L3.3-W3.3-P0.66-LS3.3-BL
- R1, R10, R11, R12, R13, R14, R15, R16, R17, R18, R19, R2, R20, R23, R26, R30, R33, R34, R37, R41, R42, R6, R7, R8, R9: footprint Resistor_SMD:R_0201_0603Metric -> Resistor_SMD:R_0402_1005Metric
- R24: value 300 -> 530; footprint Resistor_SMD:R_0201_0603Metric -> Resistor_SMD:R_0402_1005Metric
- R25, R32, R36: value 100k -> 1k
- R27: value 10k -> 1k; footprint Resistor_SMD:R_0201_0603Metric -> Resistor_SMD:R_0402_1005Metric
- R28, R35, R39, R43: value 100 -> 1k; footprint Resistor_SMD:R_0201_0603Metric -> Resistor_SMD:R_0402_1005Metric
- R31: value 100 -> 10k; footprint Resistor_SMD:R_0201_0603Metric -> Resistor_SMD:R_0402_1005Metric
- R38: value 1k -> 10k; footprint Resistor_SMD:R_0201_0603Metric -> Resistor_SMD:R_0402_1005Metric
- R40: value 100k -> 10k
- moved U12 44.3 mm to (89.7, 100.6), turned to 180 degrees
- moved D9 38.7 mm to (93.4, 103.7), turned to 90 degrees
- moved Q3 37.6 mm to (77.8, 137.8), turned to -90 degrees
- moved R16 35.8 mm to (84.2, 140.5), turned to 180 degrees
- moved D3 35.6 mm to (81.9, 140.5)
- moved R25 32.1 mm to (93.3, 92.4)
- moved P4 31.2 mm to (98.6, 120.5)
- moved P1 31.2 mm to (98.6, 89.4)
- moved R39 30.5 mm to (85.4, 119.0), turned to 180 degrees
- moved U8 29.9 mm to (89.2, 95.2), turned to 180 degrees
- moved R40 28.8 mm to (85.8, 120.7)
- moved U11 28.4 mm to (89.3, 120.8), turned to 180 degrees
- moved R33 27.1 mm to (75.0, 133.9), turned to 180 degrees
- moved U9 24.9 mm to (80.8, 136.9), turned to 90 degrees
- moved R41 24.7 mm to (86.6, 115.5), turned to 0 degrees
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- renumbered SWD to J7, LORA to U6
Connections:
- D10 pad 1: GND -> Net-(D10-K)
- D3 pad 1: GND -> Net-(D3-K)
- D6 pad 1: GND -> Net-(D6-K)
- D7 pad 1: GND -> Net-(D7-K)
- D8 pad 1: GND -> Net-(D8-K)
- D9 pad 1: GND -> Net-(D9-K)
- P1 pad 1: Net-(Q1-D) -> Net-(D8-K)
- P2 pad 1: Net-(Q9-D) -> Net-(P1-Pad2)
- P2 pad 2: Net-(P2-Pad2) -> Net-(D9-K)
- P3 pad 1: Net-(Q2-D) -> Net-(D6-K)
- P3 pad 2: Net-(P3-Pad2) -> Net-(P1-Pad2)
- P4 pad 1: Net-(Q4-D) -> Net-(P1-Pad2)
- P4 pad 2: Net-(P4-Pad2) -> Net-(D7-K)
- P5 pad 1: Net-(Q6-D) -> Net-(D3-K)
- P5 pad 2: Net-(P5-Pad2) -> Net-(P1-Pad2)
- P6 pad 1: Net-(Q12-D) -> Net-(P1-Pad2)
- P6 pad 2: Net-(P6-Pad2) -> Net-(D10-K)
- P7 pad 1: Net-(Q1-S) -> Net-(P1-Pad2)
- Q1 pad 1: Net-(Q1-G) -> Net-(Q1-S1)
- Q1 pad 2: Net-(Q1-S) -> Net-(Q1-G1)
- Q1 pad 3: Net-(Q1-D) -> Net-(Q1-S2)
- Q2 pad 1: Net-(Q2-G) -> Net-(Q2-S1)
- Q2 pad 2: Net-(Q1-S) -> Net-(Q2-G1)
- Q2 pad 3: Net-(Q2-D) -> Net-(Q2-S2)
- Q3 pad 1: Net-(Q3-G) -> Net-(Q3-S1)
- Q3 pad 2: GND -> Net-(Q3-G1)
- Q3 pad 3: Net-(Q2-G) -> Net-(Q3-S2)
- R16 pad 1: Net-(D3-A) -> Net-(P1-Pad2)
- R16 pad 2: Net-(Q9-D) -> Net-(D3-A)
- R21 pad 2: Net-(Q1-S) -> Net-(P1-Pad2)
- R24 pad 2: Net-(Q1-S) -> Net-(P1-Pad2)
- R25 pad 1: GND -> Net-(P1-Pad2)
- R25 pad 2: Net-(Q8-G) -> Net-(D8-A)
- R26 pad 1: Net-(D6-A) -> Net-(P1-Pad2)
- R26 pad 2: Net-(Q1-D) -> Net-(D6-A)
- R27 pad 1: Net-(Q1-G) -> Net-(D7-A)
- R27 pad 2: Net-(Q1-S) -> Net-(P1-Pad2)
- R28 pad 1: Net-(Q8-G) -> Net-(Q2-G1)
- R31 pad 1: Net-(Q10-G) -> Net-(Q3-G1)
- R31 pad 2: /PYRO2 -> Net-(Q3-S1)
- R32 pad 1: GND -> Net-(Q3-G1)
- R32 pad 2: Net-(Q10-G) -> /PYRO5
- R33 pad 1: Net-(Q10-D) -> Net-(Q3-G2)
- R33 pad 2: Net-(Q1-S) -> Net-(Q3-S2)
- R34 pad 1: Net-(D7-A) -> Net-(Q2-G2)
- R34 pad 2: Net-(Q2-D) -> /PYRO2
- R35 pad 1: Net-(Q3-G) -> Net-(Q1-G1)
- R36 pad 1: GND -> Net-(D9-A)
- R36 pad 2: Net-(Q3-G) -> Net-(P1-Pad2)
- R37 pad 1: Net-(Q2-G) -> Net-(Q2-G1)
- R37 pad 2: Net-(Q1-S) -> GND
- R38 pad 1: Net-(D8-A) -> GND
- R38 pad 2: Net-(Q4-D) -> Net-(Q2-G2)
- R39 pad 1: Net-(Q5-G) -> Net-(Q1-G2)
- R40 pad 2: Net-(Q5-G) -> Net-(Q1-G2)
- R41 pad 1: Net-(Q4-G) -> Net-(Q1-G1)
- R41 pad 2: Net-(Q1-S) -> GND
- R42 pad 1: Net-(D9-A) -> Net-(Q3-G2)
- R42 pad 2: Net-(Q6-D) -> /PYRO6
- R43 pad 1: Net-(Q11-G) -> Net-(D10-A)
- R43 pad 2: /PYRO5 -> Net-(P1-Pad2)
- U10 pad 2: Net-(P3-Pad2) -> Net-(Q1-S1)
- U11 pad 2: Net-(P4-Pad2) -> Net-(Q1-S2)
- U12 pad 2: Net-(P5-Pad2) -> Net-(Q2-S2)
- U13 pad 2: Net-(P6-Pad2) -> Net-(Q3-S2)
- U8 pad 2: Net-(P1-Pad2) -> Net-(Q2-S1)
- U9 pad 2: Net-(P2-Pad2) -> Net-(Q3-S1)
Routing:
- net Net-(Q1-S): track 144.5 -> 0.00 mm, vias 5 -> 0
- net Net-(P1-Pad2): track 6.96 -> 133.7 mm, vias 0 -> 3
- net /PYRO4: track 15.9 -> 58.9 mm
- net GND: track 217.3 -> 175.5 mm, vias 72 -> 62
- net Net-(D8-K): track 0.00 -> 24.2 mm
- net /PYRO1: track 48.3 -> 28.0 mm
- net Net-(D6-K): track 0.00 -> 20.3 mm
- net Net-(D7-K): track 0.00 -> 17.5 mm
- net Net-(D9-K): track 0.00 -> 15.7 mm
- net +3.3V: track 97.5 -> 111.4 mm
- net Net-(Q12-D): track 13.8 -> 0.00 mm
- net Net-(D10-K): track 0.00 -> 12.8 mm
- net Net-(D3-K): track 0.00 -> 12.1 mm
- net Net-(Q4-D): track 11.0 -> 0.00 mm
- net Net-(Q9-D): track 11.0 -> 0.00 mm
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Other:
- board text added: "${REFERENCE}"

Commit message: Update with latest changes
Parts:
- moved R19 0.65 mm to (57.0, 113.7)
- moved R14 0.13 mm to (62.9, 80.3)
- moved R6 0.10 mm to (62.8, 128.5)
Routing:
- net /POWER_ST: track 55.7 -> 53.8 mm, vias 3 -> 2
- net VBUS: track 71.2 -> 72.7 mm
- net GND: track 175.5 -> 176.1 mm, vias 62 -> 128
- net /SD_CD: track 22.5 -> 23.1 mm
Other:
- board text added: "3.3V"
- board text added: "5V"
- board text removed: "${REFERENCE}"

Commit message: Update with latest changes
Routing:
- net GND: vias 128 -> 158
Changed lines of the file:
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@@
+	)
+	(via
+		(at 103.09 145.39)
+		(size 0.6)
+		(drill 0.3)
+		(layers "F.Cu" "B.Cu")
+		(free yes)
+		(net 5)
+	)
+	(via
+		(at 86.31 149.36)
+		(size 0.6)
+		(drill 0.3)
+		(layers "F.Cu" "B.Cu")
+		(free yes)
+		(net 5)
 	)
 	(via
@@
 	)
 	(via
+		(at 41.549 133.18)
+		(size 0.6)
+		(drill 0.3)
+		(layers "F.Cu" "B.Cu")
+		(free yes)
+		(net 5)
+	)
+	(via
 		(at 53.06 102.61)
 		(size 0.6)
@@
 	)
 	(via
+		(at 68.48 44.34)
+		(size 0.6)
+		(drill 0.3)
+		(layers "F.Cu" "B.Cu")
+		(free yes)
+		(net 5)
+	)
+	(via
 		(at 88.65 103.77)
 		(size 0.6)
@@
 	)
 	(via
+		(at 103.26 75.08)
+		(size 0.6)
+		(drill 0.3)
+		(layers "F.Cu" "B.Cu")
+		(free yes)
+		(net 5)
+	)
+	(via
 		(at 43 71.1)
 		(size 0.45)
@@
 	)
 	(via
+		(at 102.82 98.13)
+		(size 0.6)
+		(drill 0.3)
+		(layers "F.Cu" "B.Cu")
+		(free yes)
+		(net 5)
+	)
+	(via
 		(at 71.55 125.14)
 		(size 0.6)
@@
 	)
 	(via
+		(at 103.12 110.49)
+		(size 0.6)
+		(drill 0.3)
+		(layers "F.Cu" "B.Cu")
+		(free yes)
+		(net 5)
+	)
+	(via
 		(at 61 90.1)
 		(size 0.45)
@@
 	)
 	(via
+		(at 40.41 58.96)
+		(size 0.6)
+		(drill 0.3)
+		(layers "F.Cu" "B.Cu")
+		(free yes)
+		(net 5)
+	)
+	(via
 		(at 72.14 124.56)
 		(size 0.6)
@@
 		(drill 0.3)
 		(layers "F.Cu" "B.Cu")
+		(net 5)
+	)
+	(via
+		(at 62.15 44.23)
+		(size 0.6)
+		(drill 0.3)
+		(layers "F.Cu" "B.Cu")
+		(free yes)
 		(net 5)
 	)
@@
 	)
 	(via
+		(at 74.23 44.37)
+		(size 0.6)
+		(drill 0.3)
+		(layers "F.Cu" "B.Cu")
+		(free yes)
+		(net 5)
+	)
+	(via
 		(at 53.9 75.7)
 		(size 0.6)
@@
 	)
 	(via
+		(at 40.175 124.7)
+		(size 0.6)
+		(drill 0.3)
+		(layers "F.Cu" "B.Cu")
+		(free yes)
+		(net 5)
+	)
+	(via
 		(at 76.04 46.8)
 		(size 0.6)
@@
 	)
 	(via
+		(at 55.24 44.34)
+		(size 0.6)
+		(drill 0.3)
+		(layers "F.Cu" "B.Cu")
+		(free yes)
+		(net 5)
+	)
+	(via
 		(at 77.45 122.75)
 		(size 0.6)
@@
 	)
 	(via
+		(at 102.85 81.62)
+		(size 0.6)
+		(drill 0.3)
+		(layers "F.Cu" "B.Cu")
+		(free yes)
+		(net 5)
+	)
+	(via
 		(at 74.7 64.9)
 		(size 0.45)
@@
 	)
 	(via
+		(at 102.24 138.13)
+		(size 0.6)
+		(drill 0.3)
+		(layers "F.Cu" "B.Cu")
+		(free yes)
+		(net 5)
+	)
+	(via
 		(at 84.78 104.76)
 		(size 0.6)
@@
 	)
 	(via
+		(at 41.62 73.09)
+		(size 0.6)
+		(drill 0.3)
+		(layers "F.Cu" "B.Cu")
+		(free yes)
+		(net 5)
+	)
+	(via
+		(at 42.08 99.23)
+		(size 0.6)
+		(drill 0.3)
+		(layers "F.Cu" "B.Cu")
+		(free yes)
+		(net 5)
+	)
+	(via
 		(at 62.88 67)
 		(size 0.45)
@@
 	)
 	(via
+		(at 103.21 50.24)
+		(size 0.6)
+		(drill 0.3)
+		(layers "F.Cu" "B.Cu")
+		(free yes)
+		(net 5)
+	)
+	(via
+		(at 49.52 44.31)
+		(size 0.6)
+		(drill 0.3)
+		(layers "F.Cu" "B.Cu")
+		(free yes)
+		(net 5)
+	)
+	(via
 		(at 69.38 60.31)
 		(size 0.6)
@@
 	)
 	(via
+		(at 40.56 117.59)
+		(size 0.6)
+		(drill 0.3)
+		(layers "F.Cu" "B.Cu")
+		(free yes)
+		(net 5)
+	)
+	(via
 		(at 48.8 47.8)
 		(size 0.6)
@@
 	)
 	(via
+		(at 41.42 145.13)
+		(size 0.6)
+		(drill 0.3)
+		(layers "F.Cu" "B.Cu")
+		(free yes)
+		(net 5)
+	)
+	(via
 		(at 60.74 140.3)
 		(size 0.6)
@@
 	)
 	(via
+		(at 102.75 63.06)
+		(size 0.6)
+		(drill 0.3)
+		(layers "F.Cu" "B.Cu")
+		(free yes)
+		(net 5)
+	)
+	(via
 		(at 67.01 46.29)
 		(size 0.6)
@@
 	(via
 		(at 90.33 71.87)
+		(size 0.6)
+		(drill 0.3)
+		(layers "F.Cu" "B.Cu")
+		(free yes)
+		(net 5)
+	)
+	(via
+		(at 97.24 151.03)
 		(size 0.6)
 		(drill 0.3)
@@
 	)
 	(via
+		(at 102.21 89.81)
+		(size 0.6)
+		(drill 0.3)
+		(layers "F.Cu" "B.Cu")
+		(free yes)
+		(net 5)
+	)
+	(via
 		(at 54.52 116.85)
 		(size 0.6)
@@
 	)
 	(via
+		(at 89.08 44.42)
+		(size 0.6)
+		(drill 0.3)
+		(layers "F.Cu" "B.Cu")
+		(free yes)
+		(net 5)
+	)
+	(via
 		(at 52.9 130.7)
 		(size 0.6)
@@
 	)
 	(via
+		(at 102.73 69.21)
+		(size 0.6)
+		(drill 0.3)
+		(layers "F.Cu" "B.Cu")
+		(free yes)
+		(net 5)
+	)
+	(via
+		(at 102.99 117.65)
+		(size 0.6)
+		(drill 0.3)
+		(layers "F.Cu" "B.Cu")
+		(free yes)
+		(net 5)
+	)
+	(via
 		(at 75.85 120.05)
 		(size 0.6)
@@
 	)
 	(via
+		(at 40.3 49.23)
+		(size 0.6)
+		(drill 0.3)
+		(layers "F.Cu" "B.Cu")
+		(free yes)
+		(net 5)
+	)
+	(via
 		(at 64.7 105.3)
 		(size 0.45)
@@
 	)
 	(via
+		(at 75.97 149.95)
+		(size 0.6)
+		(drill 0.3)
+		(layers "F.Cu" "B.Cu")
+		(free yes)
+		(net 5)
+	)
+	(via
 		(at 67.41 53.43)
 		(size 0.6)
@@
 	)
 	(via
+		(at 40.47 62.67)
+		(size 0.6)
+		(drill 0.3)
+		(layers "F.Cu" "B.Cu")
+		(free yes)
+		(net 5)
+	)
+	(via
 		(at 74.54 61.36)
 		(size 0.6)
@@
 		(net 5)
 	)
+	(via
+		(at 40.39 110.68)
+		(size 0.6)
+		(drill 0.3)
+		(layers "F.Cu" "B.Cu")
+		(free yes)
+		(net 5)
+	)

Commit message: Update to PCB
Parts:
- added G***: LOGO, LOGO, F.Cu at (85.8, 69.9)
- added J8: Conn_01x04_Pin, Connector_JST:JST_XH_B4B-XH-AM_1x04_P2.50mm_Vertical, F.Cu at (42.2, 143.2)
- moved J5 59.0 mm to (101.3, 140.4), turned to -90 degrees
- moved P7 3.61 mm to (98.6, 132.0)
- moved C16 0.78 mm to (78.3, 63.7)
- moved C17 0.78 mm to (75.3, 64.6)
- moved U3 0.78 mm to (77.8, 66.0)
Routing:
- net /S4_PWM: track 69.5 -> 93.4 mm
- net /S3_PWM: track 67.6 -> 85.8 mm
- net /S2_PWM: track 67.9 -> 81.4 mm
- net /S1_PWM: track 68.3 -> 75.2 mm
- net +BATT: track 189.5 -> 186.6 mm
- net Net-(P1-Pad2): track 133.7 -> 131.3 mm
- net /ICM_CS: track 29.3 -> 30.2 mm
- net /ICM_SDI: track 34.0 -> 34.9 mm
- net /ICM_INT1: track 43.0 -> 43.9 mm
- net /ICM_SCK: track 30.3 -> 31.1 mm
- net /ICM_SDO: track 35.1 -> 35.9 mm
- net /ICM_INT2: track 30.6 -> 31.4 mm
Other:
- board text added: "Aries"
- board text added: "Barometer"
- board text added: "IMU"
- board text added: "Rev 1.0"

Commit message: PCB fixes
Parts:
- moved J5 25.6 mm to (126.7, 137.3)
- moved Card1 25.4 mm to (74.8, 75.9)
- moved M1 25.4 mm to (73.4, 142.6)
- moved R19 25.4 mm to (82.2, 110.6)
- moved R8 25.4 mm to (81.9, 71.5)
- moved R9 25.4 mm to (81.9, 70.4)
- moved RF1 25.4 mm to (67.9, 51.5)
- moved BUZZER1 25.4 mm to (93.7, 111.7)
- moved C1 25.4 mm to (73.2, 116.6)
- moved C10 25.4 mm to (92.2, 124.4)
- moved C11 25.4 mm to (94.3, 124.4)
- moved C15 25.4 mm to (89.9, 60.5)
- moved C16 25.4 mm to (103.5, 60.7)
- moved C17 25.4 mm to (100.5, 61.5)
- moved C18 25.4 mm to (102.4, 44.0)
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Other:
- board text added: "M1"
- board text added: "M2"
- board text added: "M3"
- board text added: "M4"
