File: Hardware/Advanced Flight Computer.kicad_sch (KiCad schematic)
At the start: 5 parts, among them U1 BMP580, U2 STM32H743VITx, U3 ICM-45686

Commit message: Added symbols, wired up some components in schematic.
Parts:
- added C1: 2.2 uf, Capacitor_SMD:C_0805_2012Metric, symbol Device:C
- added C10, C11, C3, C4, C9: 22uF, symbol Device:C
- added C12: 2.7nF, symbol Device:C
- added C13: 33pF, symbol Device:C
- added C14, C15, C16, C17, C2, C7: 100nF, symbol Device:C
- added C18: 0.1uF, symbol Device:C
- added C19, C5: 10uF, symbol Device:C
- added C6: 10nF, symbol Device:C
- added C8: OPEN, symbol Device:C
- added CN1: ATGM336H-6N-74, lcsc:COMM-SMD_18P-L10.1-W9.7-P1.1-TL_L76-LB, symbol lcsc:ATGM336H-6N-74
- added D1, D2: SK6812MINI, LED_SMD:LED_SK6812MINI_PLCC4_3.5x3.5mm_P1.75mm, symbol LED:SK6812MINI
- added L1: 5.6uH, symbol Device:L
- added L2: 3.6uH, symbol Device:L
- added L3: 47nH, symbol Device:L
- added R1, R2: 5.1K, symbol Device:R
- added R10, R11, R12, R13, R8, R9: 10K, symbol Device:R
- added R3: 100k, symbol Device:R
- added R4, R6: 22.1k, symbol Device:R
- added R5: 115.8k, symbol Device:R
- added R7: 15.8k, symbol Device:R
- added RF1: BWIPX-1-001E, lcsc:IPEX-SMD_BWIPX-1-001E, symbol lcsc:BWIPX-1-001E
- added U4: LMR51430XDDCR, lcsc:SOT-23-6_L2.9-W1.6-P0.95-LS2.8-BL, symbol lcsc:LMR51430XDDCR
- added U5: AP64501SP-13, lcsc:SOIC-8_L4.9-W3.9-P1.27-LS6.0-BL-EP-1, symbol lcsc:AP64501SP-13
- added U6: RA-02, lcsc:WIRELM-SMD_RA-02-BL, symbol lcsc:RA-02
Connections:
- net ICM_SDO: now reaches U3.1 (AP_SDO/AP_AD0)
- net ICM_CS: now reaches U3.12 (AP_CS)
- net ICM_SCK: now reaches U3.13 (AP_SCL/AP_SCLK)
- net ICM_SDI: now reaches U3.14 (AP_SDA/AP_SDIO/AP_SDI)
- net ICM_INT1: now reaches U3.4 (INT1/INT)
- net +3.3V: now reaches U3.5 (VDDIO)
- net +3.3V: now also Card1.4 (VDD), U1.1 (VDDIO), U1.10 (VDD), U3.8 (VDD), C14.1, C15.1, C16.1, C17.1, C18.1, C19.1, C3.1, C4.1, CN1.8 (VCC), L1.2, R10.1, R11.1, R12.1, R13.1, R8.1, R9.1, U6.3 (3.3V)
- net GND: now reaches U3.6 (GND)
- net GND: now also Card1.12 (GND), Card1.13 (GND), U1.3 (VSS), U1.5 (SDO), U1.6 (CSB), U1.8 (VSS), U1.9 (VSS), U2.10 (VSS), U2.19 (VSSA), U2.26 (VSS), U2.49 (VSS), U2.74 (VSS), U2.99 (VSS), USB1.1 (SHELL), USB1.2 (SHELL), USB1.3 (SHELL), USB1.4 (SHELL), USB1.A1B12 (GND), USB1.B1A12 (GND), C1.2, C10.2, C11.2, C12.2, C13.2, C14.2, C15.2, C16.2, C17.2, C18.2, C19.2, C3.2, C4.2, C5.2, C6.2, C9.2, CN1.1 (GND), CN1.10 (GND), CN1.12 (GND), D1.2 (VSS), D2.2 (VSS), R1.2, R2.2, R4.2, R6.2, RF1.2 (GND), RF1.3 (GND), U4.1 (GND), U5.7 (GND), U5.9 (EP), U6.1 (GND), U6.16 (GND), U6.2 (GND), U6.9 (GND)
- net ICM_INT2: now reaches U3.9 (INT2/FSYNC/CLKIN)
- net SD_DAT2: now reaches Card1.1 (DAT2(RSV))
- net SD_DAT2: now also R10.2
- net at Card1.10 (GND): now also Card1.11 (GND), Card1.6 (VSS)
- net SD_DAT3: now reaches Card1.2 (CDDAT3(CS))
- net SD_DAT3: now also R11.2
- net SD_CMD: now reaches Card1.3 (CMD(DI))
- net SD_CMD: now also R12.2
- net SD_CLK: now reaches Card1.5 (CLK(SCLK))
- net SD_CLK: now also R13.2
- net SD_DAT0: now reaches Card1.7 (DAT0(D0))
- net SD_DAT0: now also R8.2
- net SD_DAT1: now reaches Card1.8 (DAT1(RSV))
- net SD_DAT1: now also R9.2
- net SD_CD: now reaches Card1.9 (CD)
- net BMP_SCK: now reaches U1.2 (SCK)
- net BMP_SDI: now reaches U1.4 (SDI)
- net BMP_INT: now reaches U1.7 (INT)
- net VBUS: now reaches USB1.A4B9 (VBUS)
- net VBUS: now also USB1.B4A9 (VBUS)
- net at USB1.A5 (CC1): now also R2.1
- net USB_DP: now reaches USB1.A6 (DP1)
- net USB_DP: now also USB1.B6 (DP2)
- net USB_DN: now reaches USB1.A7 (DN1)
- net USB_DN: now also USB1.B7 (DN2)
- net at USB1.B5 (CC2): now also R1.1
- new net: C7.1, U5.1 (BST)
- new net: C7.2, L2.1, U5.8 (SW)
- new net: C2.1, U4.6 (CB)
- new net: C2.2, L1.1, R3.2, U4.2 (SW)
- new net: C13.1, R7.1, U5.6 (COMP)
- new net: C12.1, R7.2
- new net: D1.1 (DOUT), D2.3 (DIN)
- new net: C5.1, U5.2 (VIN), U5.3 (EN)
- new net: C6.1, U5.4 (SS)
- new net: C8.2, R5.2, R6.1, U5.5 (FB)
- new net: R3.1, R4.1, U4.4 (FB)
- new net: CN1.14 (VCC_RF), L3.1
- new net: CN1.11 (RF_IN), L3.2, RF1.1 (SIG)
- new net +5V: C10.1, C11.1, C8.1, C9.1, D1.4 (VDD), D2.4 (VDD), L2.2, R5.1
- new net +BATT: C1.1, U4.3 (VIN), U4.5 (EN)
- new net GPS_1PPS: CN1.4 (1PPS)
- new net GPS_RXD0: CN1.3 (RXD0)
- new net GPS_TXD0: CN1.2 (TXD0)
- new net RF_DIO0: U6.5 (DIO0)
- new net RF_DIO1: U6.6 (DIO1)
- new net RF_DIO2: U6.7 (DIO2)
- new net RF_DIO3: U6.8 (DIO3)
- new net RF_DIO4: U6.10 (DIO4)
- new net RF_DIO5: U6.11 (DIO5)
- new net RF_MISO: U6.13 (MISO)
- new net RF_MOSI: U6.14 (MOSI)
- new net RF_NSS: U6.15 (NSS)
- new net RF_RESET: U6.4 (RESET)
- new net RF_SCK: U6.12 (SCK)
- new net RGB_DIN: D1.3 (DIN)
- no-connect marks 0 -> 11
Other:
- moved on the sheet: Card1, U1, U2, U3, USB1

Commit message: Update with latest changes
Parts:
- added BUZZER1: MLT-7525, lcsc:BUZ-SMD_4P-L7.5-W7.5-P7.59-TL, symbol lcsc:MLT-7525
- added C20, C21, C22, C23, C24, C25, C26: 100nF, symbol Device:C
- added C27: 10pF, symbol Device:C
- added C28, C29: 2.2uF, symbol Device:C
- added C30, C33: 1uF, symbol Device:C
- added C31, C32: 100nF, 100nF, symbol Device:C
- added C34: 22nF, symbol Device:C
- added C36: 4.7uF, symbol Device:C
- added C37, C39: 20pF, symbol Device:C
- added C38, C40: 6.8pF, symbol Device:C
- added D3, D6: LED, LED_SMD:LED_0603_1608Metric, symbol Device:LED
- added D4, D5: LED, symbol Device:LED
- added J1: Conn_01x03_Pin, Connector_PinHeader_1.00mm:PinHeader_1x03_P1.00mm_Vertical, symbol Connector:Conn_01x03_Pin
- added L4: FCM1608KF-601T03, lcsc:L0603, symbol lcsc:FCM1608KF-601T03
- added M1, M2, M3, M4, M5, M6: Motor_Servo, Connector_PinHeader_2.54mm:PinHeader_1x03_P2.54mm_Vertical, symbol Motor:Motor_Servo
- added P1, P2, P3, P4, P5, P6, P7: WJ500V-5.08-2P-14-00A, lcsc:CONN-TH_2P-P5.00_WJ500V-5.08-2P, symbol lcsc:WJ500V-5.08-2P-14-00A
- added Q1, Q2, Q3, Q4, Q5, Q6: IRLML6402_C518785, lcsc:SOT-23-3_L2.9-W1.3-P1.90-LS2.4-BR, symbol lcsc:IRLML6402_C518785
- added Q7: 2N2222AU, lcsc:SOT-89-3_L4.5-W2.4-P1.50-LS4.0-BR, symbol lcsc:2N2222AU
- added Q8: 2N7002LT1G, lcsc:SOT-23_L2.9-W1.3-P1.90-LS2.4-BR, symbol lcsc:2N7002LT1G
- added R14: 10K, symbol Device:R
- added R15, R18, R26: 1k, symbol Device:R
- added R16: 220, symbol Device:R
- added R17: 470, symbol Device:R
- added R19, R27, R30: 10k, symbol Device:R
- added R20: 22.1k, symbol Device:R
- added R21: 120k, symbol Device:R
- added R22: 100K, symbol Device:R
- added R23: 20K, symbol Device:R
- added R24: 300, symbol Device:R
- added R25: 100k, symbol Device:R
- added R28: 100, symbol Device:R
- added R29: 75k, symbol Device:R
- added SW1, SW2: TS-1088-AR02016, lcsc:SW-SMD_L3.9-W3.0-P4.45, symbol lcsc:TS-1088-AR02016
- added U7: TPS2121RUXR, lcsc:VQFN-HR-12_L2.5-W2.0-P0.50-BL, symbol lcsc:TPS2121RUXR
- added X1: X322525MOB4SI, lcsc:CRYSTAL-SMD_4P-L3.2-W2.5-BL, symbol lcsc:X322525MOB4SI
- added X2: Q13FC1350000400, lcsc:FC-135R_L3.2-W1.5, symbol lcsc:Q13FC1350000400
- C8: value OPEN -> 47pF
- R5: value 115.8k -> 115k
Connections:
- net BMP_SCK is gone; now on net I2C_SCL: U1.2 (SCK)
- net BMP_SDI is gone; now on net I2C_SDA: U1.4 (SDI)
- net GPS_RXD0 is gone; now on net GPS_RX: CN1.3 (RXD0)
- net GPS_TXD0 is gone; now on net GPS_TX: CN1.2 (TXD0)
- net SD_DAT0 is gone; now on net SD_D0: Card1.7 (DAT0(D0)), R8.2
- net SD_DAT1 is gone; now on net SD_D1: Card1.8 (DAT1(RSV)), R9.2
- net SD_DAT2 is gone; now on net SD_D2: Card1.1 (DAT2(RSV)), R10.2
- net SD_DAT3 is gone; now on net SD_D3: Card1.2 (CDDAT3(CS)), R11.2
- net +3.3V: now also U2.100 (VDD), U2.11 (VDD), U2.27 (VDD), U2.50 (VDD), U2.6 (VBAT), U2.75 (VDD), BUZZER1.1 (+), C20.1, C21.1, C22.1, C23.1, C24.1, C25.1, C36.1, L4.2, R16.1, R19.2, SW2.1
- net +5V: now also M1.2 (+), M2.2 (+), M3.2 (+), M4.2 (+), M5.2 (+), M6.2 (+)
- net +BATT: now also C5.1, U5.2 (VIN), U5.3 (EN), P7.2, R22.1, U7.2 (IN2); no longer C1.1, U4.3 (VIN), U4.5 (EN)
- net BMP_INT: now also U2.96 (PB9)
- net GND: now also Card1.10 (GND), Card1.11 (GND), Card1.6 (VSS), C20.2, C21.2, C22.2, C23.2, C24.2, C25.2, C26.1, C27.1, C28.1, C29.1, C30.2, C31.2, C32.1, C33.1, C34.2, C36.2, C37.2, C38.2, C39.2, C40.2, D4.1 (K), D5.1 (K), D6.1 (K), J1.3 (Pin_3), M1.3 (-), M2.3 (-), M3.3 (-), M4.3 (-), M5.3 (-), M6.3 (-), P1.2, P2.2, P3.2, P4.2, P5.2, P6.2, Q7.3 (EMITTER), Q8.2 (S), R14.2, R20.2, R23.2, R25.1, R29.1, SW1.1, U7.12 (GND), U7.3 (CP2), U7.4 (OV2), U7.5 (OV1), U7.6 (PR1), X1.2 (GND), X1.4 (GND)
- net GPS_1PPS: now also U2.42 (PE12), R18.1
- net ICM_CS: now also U2.28 (PA4)
- net ICM_INT1: now also U2.32 (PC4)
- net ICM_INT2: now also U2.33 (PC5)
- net ICM_SCK: now also U2.29 (PA5)
- net ICM_SDI: now also U2.31 (PA7)
- net ICM_SDO: now also U2.30 (PA6)
- net RF_DIO0: now also U2.46 (PB10)
- net RF_DIO1: now also U2.47 (PB11)
- net RF_MISO: now also U2.17 (PC2_C)
- net RF_MOSI: now also U2.16 (PC1)
- net RF_NSS: now also U2.90 (PB4)
- net RF_RESET: now also U2.36 (PB2)
- net RF_SCK: now also U2.52 (PB13)
- net RGB_DIN: now also U2.51 (PB12), R17.1; no longer D1.3 (DIN)
- net SD_CD: now also U2.84 (PD3)
- net SD_CLK: now also U2.80 (PC12)
- net SD_CMD: now also U2.83 (PD2)
- net USB_DN: now also U2.70 (PA11)
- net USB_DP: now also U2.71 (PA12)
- net VBUS: now also U7.7 (IN1)
- net HSE_IN: now reaches U2.12 (PH0)
- net HSE_IN: now also C37.1, X1.1 (OSC1)
- net HSE_OUT: now reaches U2.13 (PH1)
- net HSE_OUT: now also C39.1, X1.3 (OSC2)
- net RESET: now reaches U2.14 (NRST)
- net RESET: now also C26.2, SW1.2
- net at U2.20 (VREF+): now also C32.2, C33.2
- net at U2.21 (VDDA): now also C30.1, C31.1, L4.1
- net S5_PWM: now reaches U2.22 (PA0)
- net S5_PWM: now also M5.1 (PWM)
- net S6_PWM: now reaches U2.23 (PA1)
- net S6_PWM: now also M6.1 (PWM)
- net GPS_TX: now reaches U2.37 (PE7)
- net GPS_RX: now reaches U2.38 (PE8)
- net S1_PWM: now reaches U2.39 (PE9)
- net S1_PWM: now also M1.1 (PWM)
- net S2_PWM: now reaches U2.41 (PE11)
- net S2_PWM: now also M2.1 (PWM)
- net S3_PWM: now reaches U2.43 (PE13)
- net S3_PWM: now also M3.1 (PWM)
- net S4_PWM: now reaches U2.44 (PE14)
- net S4_PWM: now also M4.1 (PWM)
- net at U2.48 (VCAP): now also C28.2
- net BUZZER: now reaches U2.53 (PB14)
- net BUZZER: now also R15.1
- net POWER_ST: now reaches U2.55 (PD8)
- net POWER_ST: now also R19.1, U7.9 (ST)
- net PYRO1: now reaches U2.57 (PD10)
- net PYRO1: now also R28.2
- net PYRO2: now reaches U2.58 (PD11)
- net PYRO3: now reaches U2.59 (PD12)
- net PYRO4: now reaches U2.60 (PD13)
- net PYRO5: now reaches U2.61 (PD14)
- net PYRO6: now reaches U2.62 (PD15)
- net VBAT: now reaches U2.63 (PC6)
- net VBAT: now also R22.2, R23.1
- net SD_D0: now reaches U2.65 (PC8)
- net SD_D1: now reaches U2.66 (PC9)
- net at U2.73 (VCAP): now also C29.2
- net SD_D2: now reaches U2.78 (PC10)
- net SD_D3: now reaches U2.79 (PC11)
- net LSE_IN: now reaches U2.8 (PC14)
- net LSE_IN: now also C38.1, X2.1
- net LSE_OUT: now reaches U2.9 (PC15)
- net LSE_OUT: now also C40.1, X2.2
- net I2C_SDA: now reaches U2.93 (PB7)
- net BOOT: now reaches U2.94 (BOOT0)
- net BOOT: now also R14.1, SW2.2
- net I2C_SCL: now reaches U2.95 (PB8)
- net UART_RX: now reaches U2.97 (PE0)
- net UART_RX: now also J1.1 (Pin_1)
- net UART_TX: now reaches U2.98 (PE1)
- net UART_TX: now also J1.2 (Pin_2)
- net RF_DIO2: no longer names the net of U6.7 (DIO2)
- net RF_DIO3: no longer names the net of U6.8 (DIO3)
- net RF_DIO4: no longer names the net of U6.10 (DIO4)
- net RF_DIO5: no longer names the net of U6.11 (DIO5)
- new net: P7.1, Q1.2 (S), R21.2, R24.2, R27.2
- new net: P2.1, Q2.2 (S)
- new net: BUZZER1.2 (-), D3.1 (K), Q7.2 (COLLECTOR)
- new net: C27.2, U7.11 (SS)
- new net: D6.2 (A), R26.1
- new net: P1.1, Q1.3 (D), R26.2
- new net: Q7.1 (BASE), R15.2
- new net: C1.1, U4.3 (VIN), U4.5 (EN), U7.1 (OUT), U7.8 (OUT)
- new net: R20.1, U7.10 (ILM)
- new net: P6.1, Q6.2 (S)
- new net: R21.1, R29.2, R30.1
- new net: Q8.1 (G), R25.2, R28.1
- new net: Q1.1 (G), Q8.3 (D), R27.1
- new net: D3.2 (A), R16.2
- new net: D5.2 (A), R24.1
- new net: D4.2 (A), R18.2
- new net: P4.1, Q4.2 (S)
- new net: P5.1, Q5.2 (S)
- new net: P3.1, Q3.2 (S)
- new net: D1.3 (DIN), R17.2
- new net ARM_DET: C34.1, R30.2
- no-connect marks 11 -> 20
Other:
- title: (none) -> Fligth Computer
- moved on the sheet: C1, C10, C11, C12, C13, C14, C15, C16, C17, C18, C19, C2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

Commit message: Update with latest changes
Parts:
- removed Q3, Q5: IRLML6402_C518785, lcsc:SOT-23-3_L2.9-W1.3-P1.90-LS2.4-BR, symbol lcsc:IRLML6402_C518785
- added D10, D7, D8, D9: LED, LED_SMD:LED_0402_1005Metric, symbol Device:LED
- added J2: Conn_01x04_Pin, Connector_PinHeader_2.54mm:PinHeader_1x04_P2.54mm_Vertical, symbol Connector:Conn_01x04_Pin
- added J3, J4: Conn_01x02_Pin, Connector_PinHeader_2.54mm:PinHeader_1x02_P2.54mm_Vertical, symbol Connector:Conn_01x02_Pin
- added J5, J6: Conn_01x02_Pin, Connector_JST:JST_XH_B2B-XH-AM_1x02_P2.50mm_Vertical, symbol Connector:Conn_01x02_Pin
- added P8: WJ500V-5.08-2P-14-00A, lcsc:CONN-TH_2P-P5.00_WJ500V-5.08-2P, symbol lcsc:WJ500V-5.08-2P-14-00A
- added Q10, Q11, Q13, Q3, Q5: 2N7002LT1G, lcsc:SOT-23_L2.9-W1.3-P1.90-LS2.4-BR, symbol lcsc:2N7002LT1G
- added Q12, Q9: IRLML6402_C518785, lcsc:SOT-23-3_L2.9-W1.3-P1.90-LS2.4-BR, symbol lcsc:IRLML6402_C518785
- added R31, R35, R39, R43, R47: 100, Resistor_SMD:R_0201_0603Metric, symbol Device:R
- added R32, R36, R40, R44, R48: 100k, Resistor_SMD:R_0402_1005Metric, symbol Device:R
- added R33, R37, R41, R45, R49: 10k, Resistor_SMD:R_0201_0603Metric, symbol Device:R
- added R34, R38, R42, R46: 1k, Resistor_SMD:R_0201_0603Metric, symbol Device:R
- added R50, R51: 10k, Resistor_SMD:R_0402_1005Metric, symbol Device:R
- added U10, U11, U12, U13, U8, U9: 0438006.WRGT, lcsc:F0603, symbol lcsc:0438006.WRGT
- C10, C11, C3, C4, C5, C6, C8, C9: footprint (none) -> Capacitor_SMD:C_0805_2012Metric
- C12, C13, C2, C7: footprint (none) -> Capacitor_SMD:C_0603_1608Metric
- C14, C15, C16, C17, C18, C19, C20, C21, C22, C23, C24, C25, C26, C27, C28, C29, C30, C33, C34, C36, C37, C39: footprint (none) -> Capacitor_SMD:C_0402_1005Metric
- C31, C32: footprint 100nF -> Capacitor_SMD:C_0402_1005Metric
- C38, C40: value 6.8pF -> 20pF; footprint (none) -> Capacitor_SMD:C_0402_1005Metric
- D3, D6: footprint LED_SMD:LED_0603_1608Metric -> LED_SMD:LED_0402_1005Metric
- D4: footprint (none) -> LED_SMD:LED_0402_1005Metric
- D5: footprint (none) -> LED_SMD:LED_0603_1608Metric
- J1: footprint Connector_PinHeader_1.00mm:PinHeader_1x03_P1.00mm_Vertical -> Connector_PinHeader_2.54mm:PinHeader_1x03_P2.54mm_Vertical
- L1: footprint (none) -> Inductor_SMD:L_Bourns_SRP5030T; LCSC (none) -> C46595886
- L2: footprint (none) -> Inductor_SMD:L_Cenker_CKCS8040; LCSC (none) -> C223037
- L3: footprint (none) -> Inductor_SMD:L_0603_1608Metric_Pad1.05x0.95mm_HandSolder; LCSC (none) -> C98076
- R1, R10, R11, R12, R13, R14, R15, R17, R18, R19, R2, R20, R24, R26, R27, R28, R30, R6, R7, R8, R9: footprint (none) -> Resistor_SMD:R_0201_0603Metric
- R16: value 220 -> 1k; footprint (none) -> Resistor_SMD:R_0201_0603Metric
- R21, R25, R29, R3, R4, R5: footprint (none) -> Resistor_SMD:R_0402_1005Metric
- R22: value 100K -> 200K; footprint (none) -> Resistor_SMD:R_0402_1005Metric
- R23: value 20K -> 40K; footprint (none) -> Resistor_SMD:R_0201_0603Metric
Connections:
- net +3.3V: now also CN1.6 (VBAT), J2.1 (Pin_1), J5.1 (Pin_1), R50.2, R51.2; no longer R16.1
- net +5V: now also J6.1 (Pin_1)
- net +BATT: now also P8.1
- net ARM_DET: now also U2.56 (PD9)
- net GND: now also D3.1 (K), D10.1 (K), D7.1 (K), D8.1 (K), D9.1 (K), J2.2 (Pin_2), J3.1 (Pin_1), J4.1 (Pin_1), J5.2 (Pin_2), J6.2 (Pin_2), P8.2, Q10.2 (S), Q11.2 (S), Q13.2 (S), Q3.2 (S), Q5.2 (S), R32.1, R36.1, R40.1, R44.1, R48.1, U10.1, U11.1, U12.1, U13.1, U8.1, U9.1; no longer P1.2, P2.2, P3.2, P4.2, P5.2, P6.2
- net I2C_SCL: now also U2.92 (PB6), J2.3 (Pin_3); no longer U2.95 (PB8)
- net I2C_SDA: now also J2.4 (Pin_4)
- net PYRO2: now also R31.2
- net PYRO3: now also R35.2
- net PYRO4: now also R39.2
- net PYRO5: now also R43.2
- net PYRO6: now also R47.2
- net VBAT: now also U2.35 (PB1); no longer U2.63 (PC6)
- net at P7.1, Q1.2 (S), R21.2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: now also Q2.2 (S), Q4.2 (S), Q6.2 (S), Q12.2 (S), Q9.2 (S), R33.2, R37.2, R41.2, R45.2, R49.2
- net at Q2.1 (G): now also Q3.3 (D), R37.1
- net at P2.1: now also R16.2, Q9.3 (D); no longer Q2.2 (S)
- net at Q2.3 (D): now also P3.1, R34.2
- net at BUZZER1.2 (-), Q7.2 (COLLECTOR): no longer D3.1 (K)
- net at P6.1: now also Q12.3 (D), R46.2; no longer Q6.2 (S)
- net at D3.2 (A): now also R16.1; no longer R16.2
- net TH0: now reaches U2.15 (PC0)
- net TH0: now also J3.2 (Pin_2), R50.1
- net TH1: now reaches U2.24 (PA2)
- net TH1: now also J4.2 (Pin_2), R51.1
- net at Q4.1 (G): now also Q5.3 (D), R41.1
- net at P4.1: now also Q4.3 (D), R38.2; no longer Q4.2 (S)
- net at P5.1: now also Q6.3 (D), R42.2
- net at Q6.1 (G): now also Q11.3 (D), R45.1
- new net: Q11.1 (G), R43.1, R44.2
- new net: P6.2, U13.2
- new net: Q10.1 (G), R31.1, R32.2
- new net: P3.2, U10.2
- new net: Q10.3 (D), Q9.1 (G), R33.1
- new net: P5.2, U12.2
- new net: P2.2, U9.2
- new net: P4.2, U11.2
- new net: Q13.1 (G), R47.1, R48.2
- new net: D8.2 (A), R38.1
- new net: D10.2 (A), R46.1
- new net: D7.2 (A), R34.1
- new net: P1.2, U8.2
- new net: Q12.1 (G), Q13.3 (D), R49.1
- new net: Q5.1 (G), R39.1, R40.2
- new net: Q3.1 (G), R35.1, R36.2
- new net: D9.2 (A), R42.1
- no-connect marks 20 -> 22
Other:
- moved on the sheet: BUZZER1, C1, C10, C11, C12, C13, C2, C20, C21, C22, C23, C24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

Commit message: Update with latest changes
Parts:
- added J7: Conn_01x05_Pin, Connector_PinHeader_2.54mm:PinHeader_1x05_P2.54mm_Vertical, symbol Connector:Conn_01x05_Pin
Connections:
- net +3.3V: now also J7.4 (Pin_4)
- net GND: now also J7.3 (Pin_3)
- net RESET: now also J7.5 (Pin_5)
- net SWDIO: now reaches U2.72 (PA13)
- net SWDIO: now also J7.1 (Pin_1)
- net SWCLK: now reaches U2.76 (PA14)
- net SWCLK: now also J7.2 (Pin_2)

Commit message: Update with latest changes
Parts:
- removed Q1, Q12, Q2, Q4, Q6, Q9: IRLML6402_C518785, lcsc:SOT-23-3_L2.9-W1.3-P1.90-LS2.4-BR, symbol lcsc:IRLML6402_C518785
- removed Q10, Q11, Q13, Q3, Q5, Q8: 2N7002LT1G, lcsc:SOT-23_L2.9-W1.3-P1.90-LS2.4-BR, symbol lcsc:2N7002LT1G
- removed R44, R48: 100k, Resistor_SMD:R_0402_1005Metric, symbol Device:R
- removed R45, R49: 10k, Resistor_SMD:R_0201_0603Metric, symbol Device:R
- removed R46: 1k, Resistor_SMD:R_0201_0603Metric, symbol Device:R
- removed R47: 100, Resistor_SMD:R_0201_0603Metric, symbol Device:R
- added Q1, Q2, Q3: SI7232DN-T1-GE3, lcsc:POWER-1212-8_L3.3-W3.3-P0.66-LS3.3-BL, symbol lcsc:SI7232DN-T1-GE3
- R1, R10, R11, R12, R13, R14, R15, R16, R17, R18, R19, R2, R20, R23, R26, R30, R33, R34, R37, R41, R42, R6, R7, R8, R9: footprint Resistor_SMD:R_0201_0603Metric -> Resistor_SMD:R_0402_1005Metric
- R24: value 300 -> 530; footprint Resistor_SMD:R_0201_0603Metric -> Resistor_SMD:R_0402_1005Metric
- R25, R32, R36: value 100k -> 1k
- R27: value 10k -> 1k; footprint Resistor_SMD:R_0201_0603Metric -> Resistor_SMD:R_0402_1005Metric
- R28, R35, R39, R43: value 100 -> 1k; footprint Resistor_SMD:R_0201_0603Metric -> Resistor_SMD:R_0402_1005Metric
- R31: value 100 -> 10k; footprint Resistor_SMD:R_0201_0603Metric -> Resistor_SMD:R_0402_1005Metric
- R38: value 1k -> 10k; footprint Resistor_SMD:R_0201_0603Metric -> Resistor_SMD:R_0402_1005Metric
- R40: value 100k -> 10k
Connections:
- net GND: now also R37.2, R38.1, R41.2; no longer D10.1 (K), D3.1 (K), D6.1 (K), D7.1 (K), D8.1 (K), D9.1 (K), R25.1, R32.1, R36.1
- net PYRO2: now also R34.2; no longer R31.2
- net PYRO5: now also R32.2; no longer R43.2
- net PYRO6: now also R42.2
- net at R43.1: now also D10.2 (A)
- net at P7.1, R21.2, R24.2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: now also P1.2, P2.1, P3.2, P4.1, P5.2, P6.1, R16.1, R25.1, R26.1, R36.2, R43.2; no longer R33.2, R37.2, R41.2
- net at R37.1: now also R28.1, Q2.2 (G1)
- net at D6.2 (A): now also R26.2; no longer R26.1
- net at P1.1: now also D8.1 (K), Q2.7 (D1), Q2.8 (D1); no longer R26.2
- net at U13.2: now also R33.2, Q3.3 (S2); no longer P6.2
- net at R31.1: now also R32.1, Q3.2 (G1); no longer R32.2
- net at R41.1: now also R35.1, Q1.2 (G1)
- net at D3.2 (A): now also R16.2; no longer R16.1
- net at P3.1: now also D6.1 (K), Q1.7 (D1), Q1.8 (D1); no longer R34.2
- net at U10.2: now also Q1.1 (S1); no longer P3.2
- net at R33.1: now also R42.1, Q3.4 (G2)
- net at P5.1: now also D3.1 (K), Q3.7 (D1), Q3.8 (D1); no longer R42.2
- net at U12.2: now also Q2.3 (S2); no longer P5.2
- net at U9.2: now also R31.2, Q3.1 (S1); no longer P2.2
- net at R25.2: now also D8.2 (A); no longer R28.1
- net at R27.1: now also D7.2 (A)
- net at R38.2: now also R34.1, Q2.4 (G2); no longer P4.1
- net at U11.2: now also Q1.3 (S2); no longer P4.2
- net at U8.2: now also Q2.1 (S1); no longer P1.2
- net at R39.1, R40.2: now also Q1.4 (G2)
- net at D9.2 (A): now also R36.1; no longer R42.1
- new net: D7.1 (K), P4.2, Q1.5 (D2), Q1.6 (D2)
- new net: D10.1 (K), P6.2, Q3.5 (D2), Q3.6 (D2)
- new net: D9.1 (K), P2.2, Q2.5 (D2), Q2.6 (D2)
Other:
- moved on the sheet: U10

Commit message: Update to Render, PCB and Schematic
Parts:
- added J8: Conn_01x04_Pin, Connector_JST:JST_XH_B4B-XH-AM_1x04_P2.50mm_Vertical, symbol Connector:Conn_01x04_Pin
Connections:
- net S1_PWM: now also J8.1 (Pin_1)
- net S2_PWM: now also J8.2 (Pin_2)
- net S3_PWM: now also J8.3 (Pin_3)
- net S4_PWM: now also J8.4 (Pin_4)
Changed lines of the file:
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@@
 	(wire
 		(pts
+			(xy 288.29 152.4) (xy 288.29 167.64)
+		)
+		(stroke
+			(width 0)
+			(type default)
+		)
+	)
+	(wire
+		(pts
 			(xy 365.76 232.41) (xy 368.3 232.41)
 		)
@@
 	(wire
 		(pts
+			(xy 307.34 152.4) (xy 307.34 157.48)
+		)
+		(stroke
+			(width 0)
+			(type default)
+		)
+	)
+	(wire
+		(pts
 			(xy 243.84 106.68) (xy 255.27 106.68)
 		)
@@
 	(wire
 		(pts
+			(xy 304.8 152.4) (xy 304.8 157.48)
+		)
+		(stroke
+			(width 0)
+			(type default)
+		)
+	)
+	(wire
+		(pts
 			(xy 123.19 201.93) (xy 123.19 207.01)
 		)
@@
 	(wire
 		(pts
+			(xy 309.88 152.4) (xy 325.12 152.4)
+		)
+		(stroke
+			(width 0)
+			(type default)
+		)
+	)
+	(wire
+		(pts
 			(xy 29.21 233.68) (xy 34.29 233.68)
 		)
@@
 	(wire
 		(pts
+			(xy 325.12 152.4) (xy 325.12 167.64)
+		)
+		(stroke
+			(width 0)
+			(type default)
+		)
+	)
+	(wire
+		(pts
 			(xy 99.06 198.12) (xy 105.41 198.12)
 		)
@@
 	(wire
 		(pts
+			(xy 304.8 157.48) (xy 300.99 157.48)
+		)
+		(stroke
+			(width 0)
+			(type default)
+		)
+	)
+	(wire
+		(pts
 			(xy 349.25 157.48) (xy 349.25 167.64)
 		)
@@
 	(wire
 		(pts
+			(xy 307.34 157.48) (xy 312.42 157.48)
+		)
+		(stroke
+			(width 0)
+			(type default)
+		)
+	)
+	(wire
+		(pts
 			(xy 379.73 208.28) (xy 372.11 208.28)
 		)
@@
 	(wire
 		(pts
-			(xy 325.12 157.48) (xy 325.12 167.64)
-		)
-		(stroke
-			(width 0)
-			(type default)
-		)
-	)
-	(wire
-		(pts
 			(xy 379.73 228.6) (xy 379.73 208.28)
 		)
@@
 	(wire
 		(pts
-			(xy 288.29 157.48) (xy 288.29 167.64)
-		)
-		(stroke
-			(width 0)
-			(type default)
-		)
-	)
-	(wire
-		(pts
 			(xy 46.99 30.48) (xy 46.99 33.02)
 		)
@@
 	(wire
 		(pts
+			(xy 302.26 152.4) (xy 288.29 152.4)
+		)
+		(stroke
+			(width 0)
+			(type default)
+		)
+	)
+	(wire
+		(pts
 			(xy 137.16 41.91) (xy 137.16 43.18)
 		)
@@
 					(unit 1)
 				)
+			)
+		)
+	)
+	(symbol
+		(lib_id "Connector:Conn_01x04_Pin")
+		(at 304.8 157.48 90)
+		(unit 1)
+		(exclude_from_sim no)
+		(in_bom yes)
+		(on_board yes)
+		(dnp no)
+		(fields_autoplaced yes)
+		(property "Reference" "J8"
+			(at 306.07 160.02 90)
+			(effects
+				(font
+					(size 1.27 1.27)
+				)
+			)
+		)
+		(property "Value" "Conn_01x04_Pin"
+			(at 306.07 162.56 90)
+			(effects
+				(font
+					(size 1.27 1.27)
+				)
+			)
+		)
+		(property "Footprint" "Connector_JST:JST_XH_B4B-XH-AM_1x04_P2.50mm_Vertical"
+			(at 304.8 157.48 0)
+			(effects
+				(font
+					(size 1.27 1.27)
+				)
+				(hide yes)
+			)
+		)
+		(property "Datasheet" "~"
+			(at 304.8 157.48 0)
+			(effects
+				(font
+					(size 1.27 1.27)
+				)
+				(hide yes)
+			)
+		)
+		(property "Description" "Generic connector, single row, 01x04, script generated"
+			(at 304.8 157.48 0)
+			(effects
+				(font
+					(size 1.27 1.27)
+				)
+				(hide yes)
+			)
+		)
+		(pin "2"
+		)
+		(pin "1"
+		)
+		(pin "3"
+		)
+		(pin "4"
+		)
+		(instances
+			(project ""
+				(path "/622a0068-bbe7-41cd-97ce-d947c3f446e7"
+					(reference "J8")
+					(unit 1)
+				)
