File: Hardware/Advanced Flight Computer.kicad_sch (KiCad schematic)
At the start: 146 parts, among them CN1 ATGM336H-6N-74, J1 Conn_01x03_Pin, J2 Conn_01x04_Pin, J3 Conn_01x02_Pin, J4 Conn_01x02_Pin, J5 Conn_01x02_Pin, J6 Conn_01x02_Pin, J7 Conn_01x05_Pin, J8 Conn_01x04_Pin, M1 Motor_Servo, M2 Motor_Servo, M3 Motor_Servo, M4 Motor_Servo, M5 Motor_Servo, M6 Motor_Servo, P1 WJ500V-5.08-2P-14-00A, P2 WJ500V-5.08-2P-14-00A, P3 WJ500V-5.08-2P-14-00A, P4 WJ500V-5.08-2P-14-00A, P5 WJ500V-5.08-2P-14-00A, P6 WJ500V-5.08-2P-14-00A, P7 WJ500V-5.08-2P-14-00A, P8 WJ500V-5.08-2P-14-00A, Q1 SI7232DN-T1-GE3, Q2 SI7232DN-T1-GE3, Q3 SI7232DN-T1-GE3, Q7 2N2222AU, SW1 TS-1088-AR02016, SW2 TS-1088-AR02016, U1 BMP580, U10 0438006.WRGT, U11 0438006.WRGT, U12 0438006.WRGT, U13 0438006.WRGT, U2 STM32H743VITx, U3 ICM-45686, U4 LMR51430XDDCR, U5 AP64501SP-13, U6 RA-02, U7 TPS2121RUXR, U8 0438006.WRGT, U9 0438006.WRGT, X1 X322525MOB4SI, X2 Q13FC1350000400

Commit message: PCB fixes and new production file
Parts:
- added D11: LED, LED_SMD:LED_0402_1005Metric, symbol Device:LED
- added R44: 430, Resistor_SMD:R_0402_1005Metric, symbol Device:R
- R24: value 530 -> 550
Connections:
- net +BATT: now also R44.2
- net GND: now also D11.1 (K)
- new net: D11.2 (A), R44.1
